File: PCB/pomodoroPCB.kicad_pcb (KiCad board)
At the start: 2 copper layers, 40 x 26 mm, 14 parts, among them J1 Conn_01x02, J2 Conn_01x02_Female, J3 Conn_01x02, J4 Conn_01x02, J5 Conn_01x02, J6 AVR-ISP-6, J7 OLED_CONN, U1 ATmega328P-PU

Commit message: Switch from Female to Male Headers on PCB
Parts:
- J7: footprint Connector_PinSocket_2.54mm:PinSocket_1x07_P2.54mm_Vertical -> Connector_PinHeader_2.54mm:PinHeader_1x07_P2.54mm_Vertical
Changed lines of the file:
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@@
-(kicad_pcb (version 20171130) (host pcbnew "(5.1.2-1)-1")
+(kicad_pcb (version 20171130) (host pcbnew "(5.1.4-0-10_14)")
   (general
     (thickness 1.6)
@@
     (add_net "Net-(U1-Pad9)")
     (add_net VCC)
+  )
+  (module Connector_PinHeader_2.54mm:PinHeader_1x07_P2.54mm_Vertical (layer B.Cu)
+    (at 167.005 85.09 180)
+    (descr "Through hole straight pin header, 1x07, 2.54mm pitch, single row")
+    (tags "Through hole pin header THT 1x07 2.54mm single row")
+    (fp_text reference J7 (at 0 -17.78) (layer B.SilkS)
+      (effects (font (size 1 1) (thickness 0.15)) (justify mirror))
+    )
+    (fp_text value OLED_CONN (at 2.54 0.635 90) (layer B.Fab)
+      (effects (font (size 1 1) (thickness 0.15)) (justify mirror))
+    )
+    (fp_text user %R (at 0 -7.62) (layer B.Fab)
+      (effects (font (size 1 1) (thickness 0.15)) (justify mirror))
+    )
+    (fp_line (start 1.8 1.8) (end -1.8 1.8) (layer B.CrtYd) (width 0.05))
+    (fp_line (start 1.8 -17.05) (end 1.8 1.8) (layer B.CrtYd) (width 0.05))
+    (fp_line (start -1.8 -17.05) (end 1.8 -17.05) (layer B.CrtYd) (width 0.05))
+    (fp_line (start -1.8 1.8) (end -1.8 -17.05) (layer B.CrtYd) (width 0.05))
+    (fp_line (start -1.33 1.33) (end 0 1.33) (layer B.SilkS) (width 0.12))
+    (fp_line (start -1.33 0) (end -1.33 1.33) (layer B.SilkS) (width 0.12))
+    (fp_line (start -1.33 -1.27) (end 1.33 -1.27) (layer B.SilkS) (width 0.12))
+    (fp_line (start 1.33 -1.27) (end 1.33 -16.57) (layer B.SilkS) (width 0.12))
+    (fp_line (start -1.33 -1.27) (end -1.33 -16.57) (layer B.SilkS) (width 0.12))
+    (fp_line (start -1.33 -16.57) (end 1.33 -16.57) (layer B.SilkS) (width 0.12))
+    (fp_line (start -1.27 0.635) (end -0.635 1.27) (layer B.Fab) (width 0.1))
+    (fp_line (start -1.27 -16.51) (end -1.27 0.635) (layer B.Fab) (width 0.1))
+    (fp_line (start 1.27 -16.51) (end -1.27 -16.51) (layer B.Fab) (width 0.1))
+    (fp_line (start 1.27 1.27) (end 1.27 -16.51) (layer B.Fab) (width 0.1))
+    (fp_line (start -0.635 1.27) (end 1.27 1.27) (layer B.Fab) (width 0.1))
+    (pad 7 thru_hole oval (at 0 -15.24 180) (size 1.7 1.7) (drill 1) (layers *.Cu *.Mask)
+      (net 11 "Net-(J7-Pad7)"))
+    (pad 6 thru_hole oval (at 0 -12.7 180) (size 1.7 1.7) (drill 1) (layers *.Cu *.Mask)
+      (net 12 "Net-(J7-Pad6)"))
+    (pad 5 thru_hole oval (at 0 -10.16 180) (size 1.7 1.7) (drill 1) (layers *.Cu *.Mask)
+      (net 13 "Net-(J7-Pad5)"))
+    (pad 4 thru_hole oval (at 0 -7.62 180) (size 1.7 1.7) (drill 1) (layers *.Cu *.Mask)
+      (net 9 "Net-(J6-Pad3)"))
+    (pad 3 thru_hole oval (at 0 -5.08 180) (size 1.7 1.7) (drill 1) (layers *.Cu *.Mask)
+      (net 8 "Net-(J6-Pad4)"))
+    (pad 2 thru_hole oval (at 0 -2.54 180) (size 1.7 1.7) (drill 1) (layers *.Cu *.Mask)
+      (net 1 GND))
+    (pad 1 thru_hole rect (at 0 0 180) (size 1.7 1.7) (drill 1) (layers *.Cu *.Mask)
+      (net 2 VCC))
+    (model ${KISYS3DMOD}/Connector_PinHeader_2.54mm.3dshapes/PinHeader_1x07_P2.54mm_Vertical.wrl
+      (at (xyz 0 0 0))
+      (scale (xyz 1 1 1))
+      (rotate (xyz 0 0 0))
+    )
   )
   (module Connector_Wire:SolderWirePad_1x02_P3.81mm_Drill1.2mm (layer F.Cu)
@@
     )
   )
-  (module Connector_PinSocket_2.54mm:PinSocket_1x07_P2.54mm_Vertical (layer B.Cu)
-    (at 167.005 85.09 180)
-    (descr "Through hole straight socket strip, 1x07, 2.54mm pitch, single row (from Kicad 4.0.7), script generated")
-    (tags "Through hole socket strip THT 1x07 2.54mm single row")
-    (fp_text reference J7 (at 0 -17.78) (layer B.SilkS)
-      (effects (font (size 1 1) (thickness 0.15)) (justify mirror))
-    )
-    (fp_text value OLED_CONN (at 2.54 0.635 90) (layer B.Fab)
-      (effects (font (size 1 1) (thickness 0.15)) (justify mirror))
-    )
-    (fp_text user %R (at 0 -7.62) (layer B.Fab)
-      (effects (font (size 1 1) (thickness 0.15)) (justify mirror))
-    )
-    (fp_line (start -1.8 -17) (end -1.8 1.8) (layer B.CrtYd) (width 0.05))
-    (fp_line (start 1.75 -17) (end -1.8 -17) (layer B.CrtYd) (width 0.05))
-    (fp_line (start 1.75 1.8) (end 1.75 -17) (layer B.CrtYd) (width 0.05))
-    (fp_line (start -1.8 1.8) (end 1.75 1.8) (layer B.CrtYd) (width 0.05))
-    (fp_line (start 0 1.33) (end 1.33 1.33) (layer B.SilkS) (width 0.12))
-    (fp_line (start 1.33 1.33) (end 1.33 0) (layer B.SilkS) (width 0.12))
-    (fp_line (start 1.33 -1.27) (end 1.33 -16.57) (layer B.SilkS) (width 0.12))
-    (fp_line (start -1.33 -16.57) (end 1.33 -16.57) (layer B.SilkS) (width 0.12))
-    (fp_line (start -1.33 -1.27) (end -1.33 -16.57) (layer B.SilkS) (width 0.12))
-    (fp_line (start -1.33 -1.27) (end 1.33 -1.27) (layer B.SilkS) (width 0.12))
-    (fp_line (start -1.27 -16.51) (end -1.27 1.27) (layer B.Fab) (width 0.1))
-    (fp_line (start 1.27 -16.51) (end -1.27 -16.51) (layer B.Fab) (width 0.1))
-    (fp_line (start 1.27 0.635) (end 1.27 -16.51) (layer B.Fab) (width 0.1))
-    (fp_line (start 0.635 1.27) (end 1.27 0.635) (layer B.Fab) (width 0.1))
-    (fp_line (start -1.27 1.27) (end 0.635 1.27) (layer B.Fab) (width 0.1))
-    (pad 7 thru_hole oval (at 0 -15.24 180) (size 1.7 1.7) (drill 1) (layers *.Cu *.Mask)
-      (net 11 "Net-(J7-Pad7)"))
-    (pad 6 thru_hole oval (at 0 -12.7 180) (size 1.7 1.7) (drill 1) (layers *.Cu *.Mask)
-      (net 12 "Net-(J7-Pad6)"))
-    (pad 5 thru_hole oval (at 0 -10.16 180) (size 1.7 1.7) (drill 1) (layers *.Cu *.Mask)
-      (net 13 "Net-(J7-Pad5)"))
-    (pad 4 thru_hole oval (at 0 -7.62 180) (size 1.7 1.7) (drill 1) (layers *.Cu *.Mask)
-      (net 9 "Net-(J6-Pad3)"))
-    (pad 3 thru_hole oval (at 0 -5.08 180) (size 1.7 1.7) (drill 1) (layers *.Cu *.Mask)
-      (net 8 "Net-(J6-Pad4)"))
-    (pad 2 thru_hole oval (at 0 -2.54 180) (size 1.7 1.7) (drill 1) (layers *.Cu *.Mask)
-      (net 1 GND))
-    (pad 1 thru_hole rect (at 0 0 180) (size 1.7 1.7) (drill 1) (layers *.Cu *.Mask)
-      (net 2 VCC))
-    (model ${KISYS3DMOD}/Connector_PinSocket_2.54mm.3dshapes/PinSocket_1x07_P2.54mm_Vertical.wrl
-      (at (xyz 0 0 0))
-      (scale (xyz 1 1 1))
-      (rotate (xyz 0 0 0))
-    )
-  )
   (module Resistor_THT:R_Axial_DIN0207_L6.3mm_D2.5mm_P2.54mm_Vertical (layer F.Cu)
     (at 163.83 101.6 180)
@@
   (segment (start 135.89 101.6) (end 135.89 97.79) (width 0.1524) (layer F.Cu) (net 3))
   (segment (start 158.75 101.6) (end 161.29 101.6) (width 0.1524) (layer F.Cu) (net 4))
+  (segment (start 137.16 86.36) (end 133.35 90.17) (width 0.1524) (layer F.Cu) (net 5))
   (segment (start 130.81 88.9) (end 130.81 90.17) (width 0.1524) (layer F.Cu) (net 6))
   (segment (start 133.35 86.36) (end 130.81 88.9) (width 0.1524) (layer F.Cu) (net 6))
-  (segment (start 137.16 86.36) (end 133.35 90.17) (width 0.1524) (layer F.Cu) (net 5))
   (segment (start 156.845 83.185) (end 158.115 84.455) (width 0.1524) (layer B.Cu) (net 7))
   (segment (start 149.86 83.185) (end 156.845 83.185) (width 0.1524) (layer B.Cu) (net 7))
