File: PCB/pomodoroPCB.sch (KiCad schematic (older format))
At the start: 12 parts, among them J1 Conn_01x02, J2 Conn_01x02_Female, J3 Conn_01x02, J4 Conn_01x02, J5 Conn_01x02, J6 AVR-ISP-6, J7 OLED_CONN, U1 ATmega328P-PU

Commit message: Switch from Female to Male Headers on PCB
Parts:
- J7: footprint Connector_PinSocket_2.54mm:PinSocket_1x07_P2.54mm_Vertical -> Connector_PinHeader_2.54mm:PinHeader_1x07_P2.54mm_Vertical
Changed lines of the file:
@@
 F 0 "J7" H 7419 4111 50  0000 L CNN
 F 1 "OLED_CONN" H 7419 4020 50  0000 L CNN
-F 2 "Connector_PinSocket_2.54mm:PinSocket_1x07_P2.54mm_Vertical" H 7250 4050 50  0001 C CNN
+F 2 "Connector_PinHeader_2.54mm:PinHeader_1x07_P2.54mm_Vertical" H 7250 4050 50  0001 C CNN
 F 3 "~" H 7250 4050 50  0001 C CNN
 	1    7250 4050
